File: 01_Hardware/pocat-hw-main/pq_botboard/PQ_BotBoard/PQ_BotBoard.kicad_pcb (KiCad board)
At the start: 6 copper layers, 64 x 52 mm, 37 parts, among them IC1 TCN75AVOA713, J1 53261-1471, J2 Conn_01x08_MountingPin, J5 Conn_01x03_MountingPin, U1 TPS7A7002DDAR

Commit message: Pcbs actualizados corregidos (son definitivos para mandarlos a fabricar con sus respectivos Gebers en una carpeta separada)
Parts:
- removed Annotation1: GRSS, symbols-nsl:GRSS
- removed Annotation3: UPC, symbols-nsl:UPC_positiu
- removed Annotation4: Telecos, symbols-nsl:Telecos
- removed Annotation5: Bridgemaker, symbols-nsl:Bridgemaker
- removed Annotation6: snail, symbols-nsl:Snail
- added G***: LOGO, LOGO, F.Cu at (75.4, 40.1)
- added G***: LOGO, LOGO, F.Cu at (75.4, 69.6)
- added G***: LOGO, LOGO, F.Cu at (75.4, 48.1)
- added G***: LOGO, LOGO, F.Cu at (75.4, 57.1)
Other:
- board text removed: "Adriano Camps Ştefan Podaru Guillem Gràcia Solá Marc Corretgé Artur Cot Arnau Dolz Edgar Hernández Roger Almirall Júlia Alós Óscar Pavón Nil Rius Júlia Tribó"
