File: 01_Hardware/pocat-hw-main/pq_egse/EGSE.kicad_pcb (KiCad board)
At the start: 6 copper layers, 327 x 271 mm, 212 parts, among them IC1 ISL9120IRTNZ, J1 CES-110-02-L-S, J10 CES-110-02-L-S, J11 CES-110-02-L-S, J12 CES-110-02-L-S, J13 TLW-110-05-T-S, J14 TLW-110-05-T-S, J15 TLW-110-05-T-S, J16 TLW-110-05-T-S, J17 TLW-110-05-T-S, J18 TLW-110-05-T-S, J19 TLW-110-05-T-S, J2 CES-110-02-L-S, J20 TLW-110-05-T-S, J21 TLW-110-05-T-S, J22 TLW-110-05-T-S, J23 TLW-110-05-T-S, J24 HTSW-110-07-G-S, J25 SHF-105-01-L-D-TH, J26 TLW-110-05-T-S, J27 Conn_01x08_MountingPin, J28 Conn_01x08_MountingPin, J29 CES-110-02-L-S, J3 CES-110-02-L-S, J30 CES-110-02-L-S, J31 CES-110-02-L-S, J32 CES-110-02-L-S, J33 CES-110-02-L-S, J34 Conn_01x11_MountingPin, J35 Conn_01x11_MountingPin, J36 Conn_01x11_MountingPin, J37 Conn_01x11_MountingPin, J38 Conn_01x11_MountingPin, J39 53261-1471, J4 CES-110-02-L-S, J40 53261-0271, J41 Pico-Clasp_01x03, J42 TLW-108-05-T-S, J43 HTSW-110-07-G-S, J44 HTSW-110-07-G-S, J45 HTSW-110-07-G-S, J46 Conn_01x11_MountingPin, J47 Conn_01x11_MountingPin, J48 Conn_01x11_MountingPin, J49 Conn_01x11_MountingPin, J5 CES-110-02-L-S, J50 Conn_01x11_MountingPin, J51 53261-1471, J52 Pico-Clasp_01x03, J53 53261-0271, J54 73099-2, J55 73099-0, J56 CES-102-02-L-S, J57 CES-102-02-L-S, J58 SSQ-120-01-L-D, J59 CES-110-02-L-S, J6 CES-110-02-L-S, J60 CES-110-02-L-S, J61 CES-110-02-L-S, J62 68001-109HLF, J63 22-28-4153, J64 87224-2, J65 54101-S0803LF, J66 87224-2, J67 61304021021, J68 M22-2010305, J69 M22-2010305, J7 CES-110-02-L-S, J70 M22-2010305, J71 M22-2010305, J72 Conn_01x01_Socket, J73 87224-2, J8 CES-110-02-L-S, J9 CES-110-02-L-S, U1 LTC4040EUFD#PBF

Commit message: Pcbs actualizados corregidos (son definitivos para mandarlos a fabricar con sus respectivos Gebers en una carpeta separada)
Parts:
- removed the Annotation1 at (210.0, 228.0)
- removed the Annotation2 at (327.0, 100.4)
- removed Annotation4 (x2): Silkscreen_Annotation, -nsl_symbols:Telecos
- removed Annotation5 (x2): Silkscreen_Annotation, -nsl_symbols:UPC_positiu
- removed the G*** at (379.0, 100.0)
- added G***: LOGO, LOGO, F.Cu at (323.5, 308.0)
- added G***: LOGO, LOGO, F.Cu at (377.5, 103.0)
- Annotation1: footprint -nsl_symbols:Bike -> EGSE_Local:Bike__Annotation1
- Annotation1: footprint -nsl_symbols:IEEE_logo -> EGSE_Local:IEEE_logo__Annotation1
- Annotation1 (x2): footprint -nsl_symbols:Bridgemaker -> EGSE_Local:Bridgemaker__Annotation1
- Annotation2: footprint -nsl_symbols:NakNak -> EGSE_Local:NakNak__Annotation2
- Annotation2: footprint -nsl_symbols:IEEE_logo -> EGSE_Local:IEEE_logo__Annotation2
- Annotation3 (x2): footprint -nsl_symbols:NSL_long -> EGSE_Local:NSL_long__Annotation3
- C1: footprint Capacitor_SMD:C_0603_1608Metric -> EGSE_Local:C_0603_1608Metric__C1
- C2: footprint Capacitor_SMD:C_0603_1608Metric -> EGSE_Local:C_0603_1608Metric__C2
- C3: footprint Capacitor_SMD:C_1206_3216Metric -> EGSE_Local:C_1206_3216Metric__C3
- C4: footprint Capacitor_SMD:C_0603_1608Metric -> EGSE_Local:C_0603_1608Metric__C4
- C5: footprint Capacitor_SMD:C_0603_1608Metric -> EGSE_Local:C_0603_1608Metric__C5
- F1: footprint SamacSys_Parts:FUSC3116X70N -> EGSE_Local:FUSC3116X70N__F1
- G***: footprint blackcat:blackcatsmall -> EGSE_Local:blackcatsmall__G___
- H1: footprint MountingHole:MountingHole_3.2mm_M3_Pad -> EGSE_Local:MountingHole_3.2mm_M3_Pad__H1
- H10: footprint MountingHole:MountingHole_3.2mm_M3_Pad -> EGSE_Local:MountingHole_3.2mm_M3_Pad__H10
- H11: footprint MountingHole:MountingHole_3.2mm_M3_Pad -> EGSE_Local:MountingHole_3.2mm_M3_Pad__H11
- H12: footprint MountingHole:MountingHole_3.2mm_M3_Pad -> EGSE_Local:MountingHole_3.2mm_M3_Pad__H12
- H13: footprint MountingHole:MountingHole_3.2mm_M3_Pad -> EGSE_Local:MountingHole_3.2mm_M3_Pad__H13
- H14: footprint MountingHole:MountingHole_3.2mm_M3_Pad -> EGSE_Local:MountingHole_3.2mm_M3_Pad__H14
- H15: footprint MountingHole:MountingHole_3.2mm_M3_Pad -> EGSE_Local:MountingHole_3.2mm_M3_Pad__H15
- H16: footprint MountingHole:MountingHole_3.2mm_M3_Pad -> EGSE_Local:MountingHole_3.2mm_M3_Pad__H16
- H2: footprint MountingHole:MountingHole_3.2mm_M3_Pad -> EGSE_Local:MountingHole_3.2mm_M3_Pad__H2
- H3: footprint MountingHole:MountingHole_3.2mm_M3_Pad -> EGSE_Local:MountingHole_3.2mm_M3_Pad__H3
- H4: footprint MountingHole:MountingHole_3.2mm_M3_Pad -> EGSE_Local:MountingHole_3.2mm_M3_Pad__H4
- H5: footprint MountingHole:MountingHole_3.2mm_M3_Pad -> EGSE_Local:MountingHole_3.2mm_M3_Pad__H5
- H6: footprint MountingHole:MountingHole_3.2mm_M3_Pad -> EGSE_Local:MountingHole_3.2mm_M3_Pad__H6
- H61: footprint MountingHole:MountingHole_3.2mm_M3_Pad -> EGSE_Local:MountingHole_3.2mm_M3_Pad__H61
- H62: footprint MountingHole:MountingHole_3.2mm_M3_Pad -> EGSE_Local:MountingHole_3.2mm_M3_Pad__H62
- H68: footprint MountingHole:MountingHole_3.2mm_M3_Pad -> EGSE_Local:MountingHole_3.2mm_M3_Pad__H68
- H69: footprint MountingHole:MountingHole_3.2mm_M3_Pad -> EGSE_Local:MountingHole_3.2mm_M3_Pad__H69
- H7: footprint MountingHole:MountingHole_3.2mm_M3_Pad -> EGSE_Local:MountingHole_3.2mm_M3_Pad__H7
- H8: footprint MountingHole:MountingHole_3.2mm_M3_Pad -> EGSE_Local:MountingHole_3.2mm_M3_Pad__H8
- H9: footprint MountingHole:MountingHole_3.2mm_M3_Pad -> EGSE_Local:MountingHole_3.2mm_M3_Pad__H9
- J1: footprint Connector_PinSocket_2.54mm:PinSocket_1x10_P2.54mm_Vertical -> EGSE_Local:PinSocket_1x10_P2.54mm_Vertical__J1
- J10: footprint Connector_PinSocket_2.54mm:PinSocket_1x10_P2.54mm_Vertical -> EGSE_Local:PinSocket_1x10_P2.54mm_Vertical__J10
- J11: footprint Connector_PinSocket_2.54mm:PinSocket_1x10_P2.54mm_Vertical -> EGSE_Local:PinSocket_1x10_P2.54mm_Vertical__J11
- J12: footprint Connector_PinSocket_2.54mm:PinSocket_1x10_P2.54mm_Vertical -> EGSE_Local:PinSocket_1x10_P2.54mm_Vertical__J12
- J13: footprint SamacSys_Parts:HDRV10W64P0X254_1X10_2540X248X838P -> EGSE_Local:HDRV10W64P0X254_1X10_2540X248X838P__J13
- J14: footprint SamacSys_Parts:HDRV10W64P0X254_1X10_2540X248X838P -> EGSE_Local:HDRV10W64P0X254_1X10_2540X248X838P__J14
- J15: footprint SamacSys_Parts:HDRV10W64P0X254_1X10_2540X248X838P -> EGSE_Local:HDRV10W64P0X254_1X10_2540X248X838P__J15
- J16: footprint SamacSys_Parts:HDRV10W64P0X254_1X10_2540X248X838P -> EGSE_Local:HDRV10W64P0X254_1X10_2540X248X838P__J16
- J17: footprint SamacSys_Parts:HDRV10W64P0X254_1X10_2540X248X838P -> EGSE_Local:HDRV10W64P0X254_1X10_2540X248X838P__J17
- J18: footprint SamacSys_Parts:HDRV10W64P0X254_1X10_2540X248X838P -> EGSE_Local:HDRV10W64P0X254_1X10_2540X248X838P__J18
- J19: footprint SamacSys_Parts:HDRV10W64P0X254_1X10_2540X248X838P -> EGSE_Local:HDRV10W64P0X254_1X10_2540X248X838P__J19
- J2: footprint Connector_PinSocket_2.54mm:PinSocket_1x10_P2.54mm_Vertical -> EGSE_Local:PinSocket_1x10_P2.54mm_Vertical__J2
- J20: footprint SamacSys_Parts:HDRV10W64P0X254_1X10_2540X248X838P -> EGSE_Local:HDRV10W64P0X254_1X10_2540X248X838P__J20
- J21: footprint SamacSys_Parts:HDRV10W64P0X254_1X10_2540X248X838P -> EGSE_Local:HDRV10W64P0X254_1X10_2540X248X838P__J21
- J22: footprint SamacSys_Parts:HDRV10W64P0X254_1X10_2540X248X838P -> EGSE_Local:HDRV10W64P0X254_1X10_2540X248X838P__J22
- J23: footprint SamacSys_Parts:HDRV10W64P0X254_1X10_2540X248X838P -> EGSE_Local:HDRV10W64P0X254_1X10_2540X248X838P__J23
- J24: footprint SamacSys_Parts:HDRV10W64P0X254_1X10_2540X248X838P -> EGSE_Local:HDRV10W64P0X254_1X10_2540X248X838P__J24
- J25: footprint SamacSys_Parts:SHF10501LDTH -> EGSE_Local:SHF10501LDTH__J25
- J26: footprint SamacSys_Parts:HDRV10W64P0X254_1X10_2540X248X838P -> EGSE_Local:HDRV10W64P0X254_1X10_2540X248X838P__J26
- J27: footprint Connector_Molex:Molex_PicoBlade_53398-0871_1x08-1MP_P1.25mm_Vertical -> EGSE_Local:Molex_PicoBlade_53398-0871_1x08-1MP_P1.25mm_Vertical__J27
- J28: footprint Connector_Molex:Molex_PicoBlade_53398-0871_1x08-1MP_P1.25mm_Vertical -> EGSE_Local:Molex_PicoBlade_53398-0871_1x08-1MP_P1.25mm_Vertical__J28
- J29: footprint Connector_PinSocket_2.54mm:PinSocket_1x10_P2.54mm_Vertical -> EGSE_Local:PinSocket_1x10_P2.54mm_Vertical__J29
- J3: footprint Connector_PinSocket_2.54mm:PinSocket_1x10_P2.54mm_Vertical -> EGSE_Local:PinSocket_1x10_P2.54mm_Vertical__J3
- J30: footprint Connector_PinSocket_2.54mm:PinSocket_1x10_P2.54mm_Vertical -> EGSE_Local:PinSocket_1x10_P2.54mm_Vertical__J30
- J31: footprint Connector_PinSocket_2.54mm:PinSocket_1x10_P2.54mm_Vertical -> EGSE_Local:PinSocket_1x10_P2.54mm_Vertical__J31
- J32: footprint Connector_PinSocket_2.54mm:PinSocket_1x10_P2.54mm_Vertical -> EGSE_Local:PinSocket_1x10_P2.54mm_Vertical__J32
- J33: footprint Connector_PinSocket_2.54mm:PinSocket_1x10_P2.54mm_Vertical -> EGSE_Local:PinSocket_1x10_P2.54mm_Vertical__J33
- J34: footprint Connector_Molex:Molex_PicoBlade_53261-1071_1x10-1MP_P1.25mm_Horizontal -> EGSE_Local:Molex_PicoBlade_53261-1071_1x10-1MP_P1.25mm_Horizontal__J34
- J35: footprint Connector_Molex:Molex_PicoBlade_53261-1071_1x10-1MP_P1.25mm_Horizontal -> EGSE_Local:Molex_PicoBlade_53261-1071_1x10-1MP_P1.25mm_Horizontal__J35
- J36: footprint Connector_Molex:Molex_PicoBlade_53261-1071_1x10-1MP_P1.25mm_Horizontal -> EGSE_Local:Molex_PicoBlade_53261-1071_1x10-1MP_P1.25mm_Horizontal__J36
- J37: footprint Connector_Molex:Molex_PicoBlade_53261-1071_1x10-1MP_P1.25mm_Horizontal -> EGSE_Local:Molex_PicoBlade_53261-1071_1x10-1MP_P1.25mm_Horizontal__J37
- J38: footprint Connector_Molex:Molex_PicoBlade_53261-0971_1x09-1MP_P1.25mm_Horizontal -> EGSE_Local:Molex_PicoBlade_53261-0971_1x09-1MP_P1.25mm_Horizontal__J38
- J39: footprint Connector_Molex:Molex_PicoBlade_53261-1571_1x15-1MP_P1.25mm_Horizontal -> EGSE_Local:Molex_PicoBlade_53261-1571_1x15-1MP_P1.25mm_Horizontal__J39
- J4: footprint Connector_PinSocket_2.54mm:PinSocket_1x10_P2.54mm_Vertical -> EGSE_Local:PinSocket_1x10_P2.54mm_Vertical__J4
- J40: footprint Connector_Molex:Molex_PicoBlade_53261-0271_1x02-1MP_P1.25mm_Horizontal -> EGSE_Local:Molex_PicoBlade_53261-0271_1x02-1MP_P1.25mm_Horizontal__J40
- J41: footprint -nsl_connectors:Picoclasp03 -> EGSE_Local:Picoclasp03__J41
- J42: footprint SamacSys_Parts:SAMTEC_TLW-108-05-T-S -> EGSE_Local:SAMTEC_TLW-108-05-T-S__J42
- J43: footprint SamacSys_Parts:HDRV10W64P0X254_1X10_2540X248X838P -> EGSE_Local:HDRV10W64P0X254_1X10_2540X248X838P__J43
- J44: footprint SamacSys_Parts:HDRV10W64P0X254_1X10_2540X248X838P -> EGSE_Local:HDRV10W64P0X254_1X10_2540X248X838P__J44
- J45: footprint SamacSys_Parts:HDRV10W64P0X254_1X10_2540X248X838P -> EGSE_Local:HDRV10W64P0X254_1X10_2540X248X838P__J45
- J46: footprint Connector_Molex:Molex_PicoBlade_53261-1071_1x10-1MP_P1.25mm_Horizontal -> EGSE_Local:Molex_PicoBlade_53261-1071_1x10-1MP_P1.25mm_Horizontal__J46
- J47: footprint Connector_Molex:Molex_PicoBlade_53261-1071_1x10-1MP_P1.25mm_Horizontal -> EGSE_Local:Molex_PicoBlade_53261-1071_1x10-1MP_P1.25mm_Horizontal__J47
- J48: footprint Connector_Molex:Molex_PicoBlade_53261-1071_1x10-1MP_P1.25mm_Horizontal -> EGSE_Local:Molex_PicoBlade_53261-1071_1x10-1MP_P1.25mm_Horizontal__J48
- J49: footprint Connector_Molex:Molex_PicoBlade_53261-1071_1x10-1MP_P1.25mm_Horizontal -> EGSE_Local:Molex_PicoBlade_53261-1071_1x10-1MP_P1.25mm_Horizontal__J49
- J5: footprint Connector_PinSocket_2.54mm:PinSocket_1x10_P2.54mm_Vertical -> EGSE_Local:PinSocket_1x10_P2.54mm_Vertical__J5
- J50: footprint Connector_Molex:Molex_PicoBlade_53261-0971_1x09-1MP_P1.25mm_Horizontal -> EGSE_Local:Molex_PicoBlade_53261-0971_1x09-1MP_P1.25mm_Horizontal__J50
- J51: footprint Connector_Molex:Molex_PicoBlade_53261-1571_1x15-1MP_P1.25mm_Horizontal -> EGSE_Local:Molex_PicoBlade_53261-1571_1x15-1MP_P1.25mm_Horizontal__J51
- J52: footprint -nsl_connectors:Picoclasp03 -> EGSE_Local:Picoclasp03__J52
- J53: footprint Connector_Molex:Molex_PicoBlade_53261-0271_1x02-1MP_P1.25mm_Horizontal -> EGSE_Local:Molex_PicoBlade_53261-0271_1x02-1MP_P1.25mm_Horizontal__J53
- J54: footprint 73099-2:73099-2 -> EGSE_Local:73099-2__J54
- J55: footprint 73099-2:73099-2 -> EGSE_Local:73099-2__J55
- J56: footprint -nsl_connectors:CES-102-02 -> EGSE_Local:CES-102-02__J56
- J57: footprint -nsl_connectors:CES-102-02 -> EGSE_Local:CES-102-02__J57
- J58: footprint SamacSys_Parts:SSQ-120-XX-YYY-D -> EGSE_Local:SSQ-120-XX-YYY-D__J58
- J59: footprint Connector_PinSocket_2.54mm:PinSocket_1x10_P2.54mm_Vertical -> EGSE_Local:PinSocket_1x10_P2.54mm_Vertical__J59
- J6: footprint Connector_PinSocket_2.54mm:PinSocket_1x10_P2.54mm_Vertical -> EGSE_Local:PinSocket_1x10_P2.54mm_Vertical__J6
- J60: footprint Connector_PinSocket_2.54mm:PinSocket_1x10_P2.54mm_Vertical -> EGSE_Local:PinSocket_1x10_P2.54mm_Vertical__J60
- J61: footprint Connector_PinSocket_2.54mm:PinSocket_1x10_P2.54mm_Vertical -> EGSE_Local:PinSocket_1x10_P2.54mm_Vertical__J61
- J62: footprint SamacSys_Parts:HDRV9W90P0X254_1X9_2286X241X1143P -> EGSE_Local:HDRV9W90P0X254_1X9_2286X241X1143P__J62
- J63: footprint SamacSys_Parts:HDRV15W66P0X254_1X15_3810X249X838P -> EGSE_Local:HDRV15W66P0X254_1X15_3810X249X838P__J63
- J64: footprint SamacSys_Parts:872242 -> EGSE_Local:872242__J64
- J65: footprint SamacSys_Parts:54101S0803LF -> EGSE_Local:54101S0803LF__J65
- J66: footprint SamacSys_Parts:872242 -> EGSE_Local:872242__J66
- J67: footprint SamacSys_Parts:HDRRA40W64P254_2X20_5080X254X508P -> EGSE_Local:HDRRA40W64P254_2X20_5080X254X508P__J67
- J68: footprint SamacSys_Parts:HDRV3W60P0X200_1X3_600X200X525P -> EGSE_Local:HDRV3W60P0X200_1X3_600X200X525P__J68
- J69: footprint SamacSys_Parts:HDRV3W60P0X200_1X3_600X200X525P -> EGSE_Local:HDRV3W60P0X200_1X3_600X200X525P__J69
- J7: footprint Connector_PinSocket_2.54mm:PinSocket_1x10_P2.54mm_Vertical -> EGSE_Local:PinSocket_1x10_P2.54mm_Vertical__J7
- J70: footprint SamacSys_Parts:HDRV3W60P0X200_1X3_600X200X525P -> EGSE_Local:HDRV3W60P0X200_1X3_600X200X525P__J70
- J71: footprint SamacSys_Parts:HDRV3W60P0X200_1X3_600X200X525P -> EGSE_Local:HDRV3W60P0X200_1X3_600X200X525P__J71
- J72: footprint Connector_Pin:Pin_D0.9mm_L10.0mm_W2.4mm_FlatFork -> EGSE_Local:Pin_D0.9mm_L10.0mm_W2.4mm_FlatFork__J72
- J73: footprint SamacSys_Parts:872242 -> EGSE_Local:872242__J73
- J8: footprint Connector_PinSocket_2.54mm:PinSocket_1x10_P2.54mm_Vertical -> EGSE_Local:PinSocket_1x10_P2.54mm_Vertical__J8
- J9: footprint Connector_PinSocket_2.54mm:PinSocket_1x10_P2.54mm_Vertical -> EGSE_Local:PinSocket_1x10_P2.54mm_Vertical__J9
- L2: footprint Inductor_SMD:L_0805_2012Metric -> EGSE_Local:L_0805_2012Metric__L2
- R1: footprint Resistor_SMD:R_0805_2012Metric -> EGSE_Local:R_0805_2012Metric__R1
- R2: footprint Resistor_SMD:R_0603_1608Metric -> EGSE_Local:R_0603_1608Metric__R2
- R4: footprint SamacSys_Parts:ERJP03_PA3__0603_ -> EGSE_Local:ERJP03_PA3__0603___R4
- RFB1: footprint Resistor_SMD:R_0603_1608Metric -> EGSE_Local:R_0603_1608Metric__RFB1
- RFB2: footprint Resistor_SMD:R_0402_1005Metric -> EGSE_Local:R_0402_1005Metric__RFB2
- RFG1: footprint Resistor_SMD:R_0603_1608Metric -> EGSE_Local:R_0603_1608Metric__RFG1
- RFG2: footprint Resistor_SMD:R_0603_1608Metric -> EGSE_Local:R_0603_1608Metric__RFG2
- RFG3: footprint Resistor_SMD:R_0603_1608Metric -> EGSE_Local:R_0603_1608Metric__RFG3
- RFV1: footprint Resistor_SMD:R_0603_1608Metric -> EGSE_Local:R_0603_1608Metric__RFV1
- RFV2: footprint Resistor_SMD:R_0603_1608Metric -> EGSE_Local:R_0603_1608Metric__RFV2
- RFV3: footprint Resistor_SMD:R_0603_1608Metric -> EGSE_Local:R_0603_1608Metric__RFV3
- RPF1: footprint Resistor_SMD:R_0603_1608Metric -> EGSE_Local:R_0603_1608Metric__RPF1
- RPF2: footprint Resistor_SMD:R_0603_1608Metric -> EGSE_Local:R_0603_1608Metric__RPF2
- RP_CHRG1: footprint Resistor_SMD:R_0805_2012Metric -> EGSE_Local:R_0805_2012Metric__RP_CHRG1
- RP_FAULT1: footprint Resistor_SMD:R_0805_2012Metric -> EGSE_Local:R_0805_2012Metric__RP_FAULT1
- U1: footprint Package_DFN_QFN:QFN-24-1EP_4x5mm_P0.5mm_EP2.65x3.65mm -> EGSE_Local:QFN-24-1EP_4x5mm_P0.5mm_EP2.65x3.65mm__U1
- mouse-bite-2.54mm-slot (x2): footprint Panelization:mouse-bite-2.54mm-slot -> EGSE_Local:mouse-bite-2.54mm-slot__mouse-bite-2.54mm-slot
- moved Annotation2 0.63 mm to (215.0, 217.5)
