File: 01_Hardware/pocat-hw-main/pq_topboard/PQ1_TopBoard/PQ1_TopBoard.kicad_pcb (KiCad board)
At the start: 2 copper layers, 50 x 50 mm, 20 parts, among them IC1 TCN75AVUA713, J1 Conn_01x11_MountingPin

Commit message: Pcbs actualizados corregidos (son definitivos para mandarlos a fabricar con sus respectivos Gebers en una carpeta separada)
Parts:
- removed Annotation2: Silkscreen_Annotation, symbols-nsl:GRSS
- removed Annotation4: Silkscreen_Annotation, symbols-nsl:Telecos
- removed Annotation5: Silkscreen_Annotation, symbols-nsl:UPC_positiu
- added G***: LOGO, LOGO, F.Cu at (102.3, 75.8)
- added G***: LOGO, LOGO, F.Cu at (119.3, 52.8)
- added G***: LOGO, LOGO, F.Cu at (119.3, 63.8)
- added G***: LOGO, LOGO, F.Cu at (85.8, 50.3)
- moved Annotation1 22.2 mm to (85.8, 59.8), turned to 90 degrees
